File: Charge_Board.sch (KiCad schematic (older format))
At the start: 56 parts, among them J1 REF_OUT, J2 NCELL, J3 BATN_OUT, J4 Barrel_Jack, J5 Pad, J6 Pad, J7 Pad, J8 Pad, Q1 2N3904, Q2 FQP27P06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

Commit message: Added BOM
Other:
- note added: "TLO ~~ 5 C ( 40 F)\n TH1 ~~ 25.3 k\nTHI ~~ 40 C (104 F)\n TH1 ~~ 5.33 k"
- note removed: "TLO ~~ 5 C ( 40 F)\nTHI ~~ 40 C (104 F)"
Changed lines of the file:
@@
 	3800 5050 4650 5050
 Connection ~ 4650 5050
-Text Notes 3800 5250 0    50   ~ 0
-TLO ~~  5 C ( 40 F)\nTHI ~~ 40 C (104 F)
+Text Notes 3650 5400 0    50   ~ 0
+TLO ~~  5 C ( 40 F)\n   TH1 ~~ 25.3 k\nTHI ~~ 40 C (104 F)\n   TH1 ~~ 5.33 k
 $EndSCHEMATC
