File: Battery_Charger_V1.sch (KiCad schematic (older format))
At the start: 54 parts, among them Q1 SIJ482DP-T1-GE3, Q2 SIJ482DP-T1-GE3, Q3 SIJ482DP-T1-GE3, Q4 SIJ482DP-T1-GE3, U1 LTC3789, U2 AD5693, U3 OPAMP

Commit message: Updated Design
Reverted to MAX713 controller.
Design is (Mostly) a direct iteration on the master branch.
TODO: Review MAX713 behavior in presence of damaged cells.
Parts:
- removed BT?: Battery, symbol Device:Battery
- removed C17, C18, C19: 10nF, symbol Device:CP1_Small
- removed D9: BZX55B5V1, symbol Device:D_Zener_Small_ALT
- removed R15: 20k, symbol Device:R_US
- removed R16: 5.1k, symbol Device:R_US
- removed R17, R18: 3.9k, symbol Device:R_US
- removed R19: R_CFB, symbol Device:R_US
- removed U2: AD5693, Package_SO:TSSOP-10_3x3mm_P0.5mm, symbol AD5693:AD5693
- removed U3: OPAMP, symbol Simulation_SPICE:OPAMP
- added BT?: Battery, Connector:Banana_Jack_2Pin, symbol Device:Battery
- added C?: 10nF, Capacitor_THT:C_Rect_L4.0mm_W2.5mm_P2.50mm, symbol Device:C_Small
- added C? (x3): 1uF, Capacitor_THT:CP_Radial_D5.0mm_P2.00mm, symbol Device:CP1_Small
- added C? (x3): 10uF, Capacitor_THT:CP_Radial_D6.3mm_P2.50mm, symbol Device:CP1
- added D? (x2): LED, LED_THT:LED_D5.0mm, symbol Device:LED
- added J?: REF_OUT, Connector_PinHeader_2.54mm:PinHeader_1x01_P2.54mm_Vertical, symbol Connector:Conn_01x01_Female
- added J?: BATN_OUT, Connector_PinHeader_2.54mm:PinHeader_1x01_P2.54mm_Vertical, symbol Connector:Conn_01x01_Female
- added J?: NCELL, Connector_PinHeader_2.54mm:PinHeader_1x02_P2.54mm_Vertical, symbol Connector:Conn_01x02_Female
- added J? (x4): Pad, Connector:Banana_Jack_1Pin, symbol Connector:Conn_01x01_Male
- added J?: Barrel_Jack, Connector_BarrelJack:BarrelJack_CUI_PJ-102AH_Horizontal, symbol Connector:Barrel_Jack
- added NT? (x2): Net-Tie, NetTie:NetTie-2_SMD_Pad0.5mm, symbol Device:Net-Tie_2
- added NT?: Net-Tie, NetTie:NetTie-2_SMD_Pad2.0mm, symbol Device:Net-Tie_2
- added Q?: 2N3904, Package_TO_SOT_THT:TO-92_Inline, symbol Transistor_BJT:2N3904
- added Q? (x2): FQP27P06, Package_TO_SOT_THT:TO-220-3_Vertical, symbol Transistor_FET:IRF4905
- added R1: 100k, symbol Device:R_Small_US
- added R2: 280k, symbol Device:R_Small_US
- added R3: 2.7k, symbol Device:R_Small_US
- added R? (x4): 0.56, Resistor_THT:R_Axial_DIN0309_L9.0mm_D3.2mm_P12.70mm_Horizontal, symbol Device:R
- added R? (x7): 27k, Resistor_THT:R_Axial_DIN0207_L6.3mm_D2.5mm_P10.16mm_Horizontal, symbol Device:R
- added R?: 43k, Resistor_THT:R_Axial_DIN0207_L6.3mm_D2.5mm_P10.16mm_Horizontal, symbol Device:R
- added R? (x3): 18k, Resistor_THT:R_Axial_DIN0207_L6.3mm_D2.5mm_P10.16mm_Horizontal, symbol Device:R
- added R? (x2): 1k, Resistor_THT:R_Axial_DIN0207_L6.3mm_D2.5mm_P10.16mm_Horizontal, symbol Device:R
- added R?: 100k, Resistor_THT:R_Axial_DIN0207_L6.3mm_D2.5mm_P10.16mm_Horizontal, symbol Device:R
- added R? (x2): 10k, Resistor_THT:R_Axial_DIN0207_L6.3mm_D2.5mm_P10.16mm_Horizontal, symbol Device:R
- added RV?: 10k, Potentiometer_THT:Potentiometer_Bourns_PTV09A-1_Single_Vertical, symbol Device:R_POT
- added TH?: NTCLE100E3103JB0, Connector_PinHeader_2.54mm:PinHeader_1x02_P2.54mm_Vertical, symbol Device:Thermistor_NTC
- added U?: MAX713, Package_SO:SOIC-16_4.55x10.3mm_P1.27mm, symbol Battery_Management:MAX713EPE
- added U?: LM7805, Package_TO_SOT_THT:TO-220-3_Vertical, symbol Regulator_Linear:LM7805_TO220
Connections:
- net labels added: +5V, +BATT, -BATT, 2V, 5VA, CC, DC, FASTCHG_LED, FB_BATT+, FB_BATT-, FEEDBACK, GND, GNDD, PGM0, PGM1, PWR_LED, TEMP, THI, TLO, VCELL, VSMPS, Vfb, nFASTCHG
- net labels removed: Ibat, SCL, SDA, Vbat, Vdiv, Vin, Vsense
- wire segments 119 -> 197
- no-connect marks 3 -> 4
Other:
- note added: "(External)\nTemp. Sensor"
- note added: "BUCK-BOOST Converter (Feeds Battery)"
- note added: "Cascode for\nHigh Cell Count"
- note added: "Caution: HOT\nConsider Heatsink"
- note added: "Charge Controller"
- note added: "DC Supply Voltage (19v to 24v)"
- note added: "DRV Sinks Current to Increase Voltage\nDesign for a 28 V Max Output\n\nVout = (0.8 V) * (R1 + R2)/(R1)\nRegulator tries to keep Vfb at (0.8 V)\n\n(280k, 100k) Sets a Nominal 3 V Target.\n\nAt 28 V, 97 uA across R2.\nAssume V_CE (Sat) 0.5 V,\nV(R3) = 0.3 V at 97 uA --> R3 = 3.1 kOhm\nfor V_CE (Sat) 0.7 V ... R3 = 1.0 kOhm"
- note added: "ID: 4 mm\nMounting Holes"
- note added: "LP Filtered\nFeedback\n"
- note added: "Linear 5V (Feeds MAX713)"
- note added: "NiCd / NiMH Notes:"
- note added: "Ref. Cell Voltage"
- note added: "TLO ~~ 5 C ( 40 F)\n TH1 ~~ 25.3 k\nTHI ~~ 40 C (104 F)\n TH1 ~~ 5.33 k"
- note added: "[14.4 V Battery Pack]\n(12 Cells in Series)\n PGM0 -- REF\n PGM1 -- BATT-\n~~18.24 V Charged (NiMH)\n~~19.80 V Charged (NiCd)"
- note added: "[18.0 V Battery Pack]\n(15 Cells in Series)\n PGM0 -- BATT-\n PGM1 -- REF\n~~22.80 V Charged (NiMH)\n~~24.75 V Charged (NiCd)"
- note added: "[Charging Temperature]\nAbsolute (32 to 113) F\nRecommended (50 to 85) F\n\n[Cell Voltage]\n1.20 V / Cell (Nominal)\n1.52 V / Cell (NiMH, Charged)\n1.65 V / Cell (NiCd, Charged)\n(See) Figure 2.10 of https://doi.org/10.1016/B978-0-12-407947-2.00002-X\nhttps://www.sciencedirect.com/topics/engineering/open-circuit-cell-voltage"
- note added: "~~1.786 A Max\nCharge Path"
- note removed: "Clamp to ~~5V"
- moved on the sheet: C1, C10, C11, C12, C13, C14, C15, C16, C2, C3, C4, C5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

Commit message: Corrected Q1
P-Channel MOSFET was oriented incorrectly.
Parts:
- removed C16: 330 μF, symbol Device:CP1
- removed C3: 3.3 μF, symbol Device:C_Small
- removed J?: REF_OUT, Connector_PinHeader_2.54mm:PinHeader_1x01_P2.54mm_Vertical, symbol Connector:Conn_01x01_Female
- removed J?: BATN_OUT, Connector_PinHeader_2.54mm:PinHeader_1x01_P2.54mm_Vertical, symbol Connector:Conn_01x01_Female
- removed J?: NCELL, Connector_PinHeader_2.54mm:PinHeader_1x02_P2.54mm_Vertical, symbol Connector:Conn_01x02_Female
- removed R?: 0.56, Resistor_THT:R_Axial_DIN0309_L9.0mm_D3.2mm_P12.70mm_Horizontal, symbol Device:R
- added C12: 2.2 μF, symbol Device:C_Small
- added C24, C25: 270 μF, symbol Device:CP1
- added J2: Switch, symbol Connector:Conn_01x02_Male
- added JP1: PROTO, symbol Device:Jumper_NO_Small
- added R28: 27 kΩ, Resistor_THT:R_Axial_DIN0207_L6.3mm_D2.5mm_P10.16mm_Horizontal, symbol Device:R_US
- added R5: 0.56 Ω, Resistor_THT:R_Axial_DIN0309_L9.0mm_D3.2mm_P12.70mm_Horizontal, symbol Device:R_US
- added R8: 7.5 Ω, symbol Device:R_Small_US
- added SW1: (14.4 / 18.0) V Mode Switch, symbol Switch:SW_Push_DPDT
- added TP1, TP2, TP3, TP4: TestPoint_Small, symbol Connector:TestPoint_Small
- C10, C11, C9: renamed from C?; value 1uF -> 1 uF
- C17, C18, C19: renamed from C?; value 10uF -> 10 uF
- C3: renamed from C?; value 10nF -> 10 nF
- D1: renamed from D?; value LED -> Red; symbol Device:LED -> Device:LED_ALT
- D2: renamed from D?; value LED -> Yellow; symbol Device:LED -> Device:LED_ALT
- J1: renamed from J?; value Barrel_Jack -> PJ-063AH; footprint Connector_BarrelJack:BarrelJack_CUI_PJ-102AH_Horizontal -> Connector_BarrelJack:BarrelJack_CUI_PJ-063AH_Horizontal_CircularHoles
- Q1, Q2: renamed from Q?; value FQP27P06 -> IRF4905
- R12, R13: renamed from R?; value 1k -> 1 kΩ; symbol Device:R -> Device:R_US
- R16: renamed from R3; value 2.7k -> 2.7 kΩ
- R17, R18: renamed from R?; value 10k -> 10 kΩ; symbol Device:R -> Device:R_US
- R20, R21, R22: renamed from R?; value 18k -> 18 kΩ; symbol Device:R -> Device:R_US
- R23, R24, R25, R26, R27, R29: renamed from R?; value 27k -> 27 kΩ; symbol Device:R -> Device:R_US
- R3, R4, R6: renamed from R?; value 0.56 -> 0.56 Ω; symbol Device:R -> Device:R_US
- R30: renamed from R?; value 43k -> 43 kΩ; symbol Device:R -> Device:R_US
- R31: renamed from R?; value 100k -> 100 kΩ; symbol Device:R -> Device:R_US
- R33: renamed from R1; value 100k -> 100 kΩ
- R35: renamed from R?; value 27k -> 270 kΩ; symbol Device:R -> Device:R_US
- R36: renamed from R2; value 280k -> 270 kΩ
- R5: renamed from R1; value 10 Ω -> 0.56 Ω; footprint (none) -> Resistor_THT:R_Axial_DIN0309_L9.0mm_D3.2mm_P12.70mm_Horizontal
- RV1: renamed from RV?; value 10k -> 10 kΩ; symbol Device:R_POT -> Device:R_POT_US
- TH1: renamed from TH?; value NTCLE100E3103JB0 -> 10 kΩ; symbol Device:Thermistor_NTC -> Device:Thermistor_NTC_US; Model (none) -> NTCLE100E3103JB0
- gave numbers to parts that had none: 11
- renumbered C5 to C1, C12 to C13, C13 to C14, C14 to C15, C15 to C16, C7 to C2, C5 to C20, C9 to C21, C2 to C22, C1 to C23, C8 to C4, C10 to C5, C11 to C6, C4 to C7, C6 to C8, D6 to D3, D7 to D4, D1 to D5, D2 to D6, D3 to D7, D4 to D8, D8 to D9, Q1 to Q3, Q2 to Q4, Q3 to Q5, Q4 to Q6, R13 to R1, R8 to R14, R9 to R15, R2 to R19, R14 to R2, R7 to R32, R3 to R34, R12 to R7, R6 to R9, U1 to U2
Connections:
- net labels added: REF
- wire segments 197 -> 215
- no-connect marks 4 -> 1
Other:
- note added: "(+Batt) Replaced with VSMPS\nto ensure output voltage is\nalways regulated. Delta_V\nassociated with Q2 should\nbe minimal: Sub-(90 mV)."
- note added: "Cascode for High Cell Count"
- note added: "DC Supply Voltage (7.5v to 30v)"
- note added: "DRV Sinks Current to Increase Voltage\nDesign for a 28 V Max Output\n\nVout = (0.8 V) * (R1 + R2)/(R1)\nRegulator tries to keep Vfb at (0.8 V)\n\n(270k, 100k) Sets a Nominal ~~3 V Target.\n\nAt 28 V, 97 uA across R2.\nAssume V_CE (Sat) 0.5 V,\nV(R3) = 0.3 V at 97 uA --> R3 = 3.1 kOhm\nfor V_CE (Sat) 0.7 V ... R3 = 1.0 kOhm"
- note added: "PGM 2,3 Set per Table 3\nTimeout 264 min"
- note added: "[14.4 V Battery Pack]\n(12 Cells in Series)\n PGM0 -- REF\n PGM1 -- BATT-\n~~18.24 V Charged (NiMH)\n~~19.80 V Charged (NiCd)\n4.8V Under-Volt Lock-Out"
- note added: "[18.0 V Battery Pack]\n(15 Cells in Series)\n PGM0 -- BATT-\n PGM1 -- REF\n~~22.80 V Charged (NiMH)\n~~24.75 V Charged (NiCd)\n6.0V Under-Volt Lock-Out"
- note added: "~~1.8 A Max\nCharge Path"
- note removed: "Cascode for\nHigh Cell Count"
- note removed: "DC Supply Voltage (19v to 24v)"
- note removed: "DRV Sinks Current to Increase Voltage\nDesign for a 28 V Max Output\n\nVout = (0.8 V) * (R1 + R2)/(R1)\nRegulator tries to keep Vfb at (0.8 V)\n\n(280k, 100k) Sets a Nominal 3 V Target.\n\nAt 28 V, 97 uA across R2.\nAssume V_CE (Sat) 0.5 V,\nV(R3) = 0.3 V at 97 uA --> R3 = 3.1 kOhm\nfor V_CE (Sat) 0.7 V ... R3 = 1.0 kOhm"
- note removed: "[14.4 V Battery Pack]\n(12 Cells in Series)\n PGM0 -- REF\n PGM1 -- BATT-\n~~18.24 V Charged (NiMH)\n~~19.80 V Charged (NiCd)"
- note removed: "[18.0 V Battery Pack]\n(15 Cells in Series)\n PGM0 -- BATT-\n PGM1 -- REF\n~~22.80 V Charged (NiMH)\n~~24.75 V Charged (NiCd)"
- note removed: "~~1.786 A Max\nCharge Path"
- moved on the sheet: BT1, C1, C10, C11, C13, C14, C15, C16, C17, C18, C19, C2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

Commit message: Draft PCB
Minor edits to schematic.
PCB is **NOT** fully routed.
Parts:
- removed Q3, Q4, Q5, Q6: SIJ482DP-T1-GE3, symbol Device:Q_NMOS_DGS
- removed R5: 0.56 Ω, Resistor_THT:R_Axial_DIN0309_L9.0mm_D3.2mm_P12.70mm_Horizontal, symbol Device:R_Small_US
- added Q3, Q4: PSMN4R2_40VSH, Nexperia:LFPAK56D, symbol q_dual_nmos_psmn4r2_40vsh:Q_DUAL_NMOS_PSMN4R2_40VSH
- added R37: 100 kΩ, Resistor_SMD:R_0805_2012Metric_Pad1.20x1.40mm_HandSolder, symbol Device:R_Small_US
- C1, C2: footprint (none) -> Capacitor_SMD:C_0603_1608Metric_Pad1.08x0.95mm_HandSolder
- C10, C11, C9: value 1 uF -> 1 μF; footprint Capacitor_THT:CP_Radial_D5.0mm_P2.00mm -> Capacitor_SMD:C_0805_2012Metric_Pad1.18x1.45mm_HandSolder
- C12, C13, C14, C15, C16: footprint (none) -> Capacitor_SMD:C_1206_3216Metric_Pad1.33x1.80mm_HandSolder
- C17, C18, C19: footprint Capacitor_THT:CP_Radial_D6.3mm_P2.50mm -> Capacitor_SMD:C_1210_3225Metric_Pad1.33x2.70mm_HandSolder
- C20, C21: footprint (none) -> Capacitor_SMD:C_1210_3225Metric_Pad1.33x2.70mm_HandSolder
- C22, C23, C24, C25: footprint (none) -> Capacitor_THT:CP_Radial_D10.0mm_P5.00mm
- C3: footprint Capacitor_THT:C_Rect_L4.0mm_W2.5mm_P2.50mm -> Capacitor_SMD:C_0603_1608Metric_Pad1.08x0.95mm_HandSolder
- C4, C7, C8: footprint (none) -> Capacitor_SMD:C_0805_2012Metric_Pad1.18x1.45mm_HandSolder
- C5, C6: value 220 nF -> 470 nF; footprint (none) -> Capacitor_SMD:C_1206_3216Metric_Pad1.33x1.80mm_HandSolder
- D3, D4: footprint (none) -> Diode_SMD:D_PowerDI-123
- D5, D6, D7, D8: footprint (none) -> Diode_SMD:D_SMA-SMB_Universal_Handsoldering
- D9: value BAS16 -> BAV99,235; footprint (none) -> Diode_SMD:D_SOT-23_ANK; symbol Device:D_Small_ALT -> Device:D_x2_Serial_AKC
- J2: footprint (none) -> Connector_PinHeader_2.54mm:PinHeader_1x02_P2.54mm_Vertical
- J3, J4, J5, J6: footprint Connector:Banana_Jack_1Pin -> TestPoint:TestPoint_Loop_D3.80mm_Drill2.8mm
- JP1: footprint (none) -> Jumper:SolderJumper-2_P1.3mm_Open_Pad1.0x1.5mm
- L1: footprint (none) -> WE-HCF:2818
- R1, R10, R11, R14, R15, R16, R19, R2, R32, R33, R34, R36, R7, R8, R9: footprint (none) -> Resistor_SMD:R_0805_2012Metric_Pad1.20x1.40mm_HandSolder
- R12, R13, R17, R18, R20, R21, R22, R23, R24, R25, R26, R27, R28, R29, R30, R31, R35: footprint Resistor_THT:R_Axial_DIN0207_L6.3mm_D2.5mm_P10.16mm_Horizontal -> Resistor_SMD:R_0805_2012Metric_Pad1.20x1.40mm_HandSolder
- R3, R4, R5, R6: footprint Resistor_THT:R_Axial_DIN0309_L9.0mm_D3.2mm_P12.70mm_Horizontal -> Resistor_THT:R_Axial_DIN0617_L17.0mm_D6.0mm_P20.32mm_Horizontal
- SW1: footprint (none) -> Button_Switch_THT:SW_E-Switch_EG1271_DPDT
- TP1, TP2, TP3, TP4: footprint (none) -> TestPoint:TestPoint_Pad_2.5x2.5mm
Connections:
- net 2V is gone; now on net REF: R20.1, R21.2, TH1.1
- net BG2: now also D9.3 (common), Q4.2 (G2); no longer D9.2 (A)
- net DC: now also Q3.5 (D1), Q3.6 (D1), R37.2
- net GND: now also C1.1, C2.1, C20.2, C21.2, C4.1, C7.2, C8.1, R34.2, U2.12 (ILIM), U2.15 (TRIM), U2.20 (EXTVCC), U2.6 (SGND); no longer J5.1 (Pin_1), J6.1 (Pin_1)
- net TG2: now also Q4.4 (G1)
- net Vout: now also C15.1, D7.1 (K), R10.1, R2.1, Q4.5 (D1), Q4.6 (D1)
- net at R7.2, U2.19 (BG2): now also D9.2 (K); no longer D9.1 (K)
- net at D7.2 (A), D8.1 (K), L1.2: now also Q4.7 (D2), Q4.7 (S1), Q4.8 (D2), Q4.8 (S1)
- net at D6.2 (A), D8.2 (A), R1.2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: now also Q3.1 (S2), Q4.1 (S2)
- net at C5.2, D5.2 (A), D6.1 (K)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: now also Q3.7 (D2), Q3.7 (S1), Q3.8 (D2), Q3.8 (S1)
- net at C20.1, U2.10 (VINSNS): now also R37.1
- net at U2.23 (BG1): now also Q3.2 (G2)
- net at U2.26 (TG1): now also Q3.4 (G1)
- removed net GNDA: C1.1, C12.2, C15.2, C16.2, C2.1, C20.2, C21.2, C22.2, C23.2, C24.2, C25.2, C4.1, C7.2, C8.1, R1.1, R15.1, R33.2, R34.2, U2.12 (ILIM), U2.15 (TRIM), U2.20 (EXTVCC), U2.24 (PGND), U2.6 (SGND)
- net GNDD renamed GNDPWR
- net GNDPWR: now also C12.2, C15.2, C16.2, C22.2, C23.2, C24.2, C25.2, R1.1, R15.1, R33.2, U2.24 (PGND)
- no-connect marks 1 -> 5
Other:
- moved on the sheet: C15, D5, D6, J5, J6, R1, R7

Commit message: Draft PCB(3)
Pre-DRC
Connections:
- net Vfb is gone; now on net V_FB: R16.2, R33.1, R36.2
Changed lines of the file:
@@
 	7900 4250 7900 4300
 Text Label 7600 4250 2    50   ~ 0
-Vfb
+V_FB
 Text Notes 8750 4700 0    50   ~ 0
 DRV Sinks Current to Increase Voltage\nDesign for a 28 V Max Output\n\nVout = (0.8 V) * (R1 + R2)/(R1)\nRegulator tries to keep Vfb at (0.8 V)\n\n(270k, 100k) Sets a Nominal ~~3 V Target.\n\nAt 28 V, 97 uA across R2.\nAssume V_CE (Sat) 0.5 V,\nV(R3) = 0.3 V at 97 uA --> R3 = 3.1 kOhm\nfor V_CE (Sat) 0.7 V ... R3 = 1.0 kOhm

Commit message: Revised Switch Footprint
Parts:
- Q3, Q4: symbol q_dual_nmos_psmn4r2_40vsh:Q_DUAL_NMOS_PSMN4R2_40VSH -> Battery_Charger_V1-rescue:Q_DUAL_NMOS_PSMN4R2_40VSH-q_dual_nmos_psmn4r2_40vsh
- SW1: footprint Button_Switch_THT:SW_E-Switch_EG1271_DPDT -> CK_Switches:DPDT
Changed lines of the file:
@@
 F 0 "SW1" H 5950 6300 50  0000 C CNN
 F 1 "(14.4 / 18.0) V Mode Switch" H 6000 5450 50  0000 C CNN
-F 2 "Button_Switch_THT:SW_E-Switch_EG1271_DPDT" H 5950 6100 50  0001 C CNN
+F 2 "CK_Switches:DPDT" H 5950 6100 50  0001 C CNN
 F 3 "~" H 5950 6100 50  0001 C CNN
 	1    5950 5900
@@
 	8300 2400 8250 2400
 $Comp
-L q_dual_nmos_psmn4r2_40vsh:Q_DUAL_NMOS_PSMN4R2_40VSH Q3
+L Battery_Charger_V1-rescue:Q_DUAL_NMOS_PSMN4R2_40VSH-q_dual_nmos_psmn4r2_40vsh Q3
 U 1 1 6375112D
 P 8075 1450
@@
 $EndComp
 $Comp
-L q_dual_nmos_psmn4r2_40vsh:Q_DUAL_NMOS_PSMN4R2_40VSH Q3
+L Battery_Charger_V1-rescue:Q_DUAL_NMOS_PSMN4R2_40VSH-q_dual_nmos_psmn4r2_40vsh Q3
 U 2 1 6375262B
 P 8075 1850
@@
 	8100 1650 8175 1650
 $Comp
-L q_dual_nmos_psmn4r2_40vsh:Q_DUAL_NMOS_PSMN4R2_40VSH Q4
+L Battery_Charger_V1-rescue:Q_DUAL_NMOS_PSMN4R2_40VSH-q_dual_nmos_psmn4r2_40vsh Q4
 U 1 1 63775358
 P 9250 1450
@@
 $EndComp
 $Comp
-L q_dual_nmos_psmn4r2_40vsh:Q_DUAL_NMOS_PSMN4R2_40VSH Q4
+L Battery_Charger_V1-rescue:Q_DUAL_NMOS_PSMN4R2_40VSH-q_dual_nmos_psmn4r2_40vsh Q4
 U 2 1 63775F64
 P 9250 1850
